Commit message: modified xacro and urdf

File: gazebo/urdf/imu.urdf.xacro (robot description, xacro)
@@ -4,5 +4,5 @@
       <joint name="imu+quad_joint" type="fixed">
       <xacro:insert_block name="origin" />
-      <parent link="link_quad"/>
+      <parent link="chassis_link"/>
       <child link="link_imu"/>
       </joint>
@@ -11,5 +11,5 @@
      <origin xyz="0 0 0.16" rpy="0 0 0"/>
      <mass value="0.003"/>
-     <inertia ixx="100"  ixy="0"  ixz="0" iyy="100" iyz="0" izz="100" />
+     <inertia ixx="0.0001" ixy="0" ixz="0" iyy="0.0001" iyz="0" izz="0.0001" />
    </inertial>
      <visual>
@@ -32,5 +32,5 @@
       <update_rate>100</update_rate>
       <visualize>true</visualize>
-      <topic>imu_signal</topic>
+      <topic>__default_topic__</topic>
       <plugin filename="libgazebo_ros_imu_sensor.so" name="imu_plugin">
         <topicName>imu</topicName>
@@ -43,5 +43,5 @@
         <initialOrientationAsReference>false</initialOrientationAsReference>
       </plugin>
-      <pose>0 0 0 0 0 0</pose>
+      <pose>0 0 0.16 0 0 0</pose>
     </sensor>
   </gazebo>

File: gazebo/urdf/quadcopter_chassis.urdf.xacro (robot description, xacro)
@@ -3,9 +3,10 @@
   <!-- Main quadrotor link -->
   <xacro:macro name="quadrotor_chassis_macro">
-    <link name="base_link">
+    <link name="chassis_link">
      <inertial>
      <origin xyz="0 0 0.2" rpy="0 0 0"/>
      <mass value="1"/>
-     <inertia ixx="100"  ixy="0"  ixz="0" iyy="100" iyz="0" izz="100" />
+     <origin xyz="0.2 0 0" />
+     <inertia ixx="0.01152" ixy="0.0" ixz="0.0" iyy="0.01152" iyz="0.0" izz="0.0218" />
    </inertial>
    <visual>
@@ -16,5 +17,5 @@
    </visual>
    <collision>
-        <origin xyz="0 0 0" rpy="0 0 0" />
+        <origin xyz="0 0 0.2" rpy="0 0 0" />
         <geometry>
           <mesh><uri>/home/saykay/drone/gazebo/meshes/Drone_assembly1_v1.dae</uri></mesh>
